File: HW/Kicad Project/BigWater.sch (KiCad schematic (older format))
At the start: 58 parts, among them J1 Conn_01x19, J2 Conn_01x19, J3 ADS1115, J4 Conn_01x02, J5 I2C, J6 Conn_01x03, J7 StripeB, J8 StripeA, SW1 SW_SPDT, SW2 SW_Push, SW3 SW_Push, SW4 SW_Push, U1 LM7805_TO220

Commit message: Guardado progreso día lunes
Parts:
- removed J6: Conn_01x03, Connector_PinSocket_2.54mm:PinSocket_1x03_P2.54mm_Vertical, symbol Connector_Generic:Conn_01x03
- added J6: Vout, Connector_PinSocket_2.54mm:PinSocket_1x02_P2.54mm_Vertical, symbol Connector_Generic:Conn_01x02
- added R18: 145, Resistor_THT:R_Axial_DIN0207_L6.3mm_D2.5mm_P7.62mm_Horizontal, symbol Device:R
Connections:
- net 5V: now also C4.1, U1.3 (VO), J6.2 (Pin_2), R18.1; no longer D3.1 (K)
- net GND: now also D3.1 (K), J6.1 (Pin_1)
- new net: D3.2 (A), R18.2
Other:
- note added: "Para calcular ancho, calcular regimen transitorio y regimen general, hayar máximo."
- note added: "Resistencia limitante"
- note added: "Transistores de potencia. MOSFET, IGBT. Infineon (Transistores en semipuente)"
- note added: "Valor raro para THT\n"
- note added: "Ver máximo de consumo de micro y en funcion de este, ajustar el LM7805."
- moved on the sheet: C2, C7, D3, JAnalog3, JEC1, JPH1, JTDS1, JTURB1, R3, R4, R5
